Commit message: joao

File: model/ft_sensor.gazebo.xacro (robot description, xacro)
@@ -14,12 +14,12 @@
     <gazebo>
         <plugin name="${name}_ft_sensor" filename="libgazebo_ros_ft_sensor.so">
-        <updateRate>1000.0</updateRate>
+        <updateRate>100.0</updateRate>
         <topicName>${parent}_${name}/ft_sensor_topic</topicName>
         <jointName>${parent}_${name}_measure_joint</jointName>
-        <noise>
+        <!--noise>
           <type>gaussian</type>
           <mean>0.0</mean>
-          <stddev>0.003</stddev> <!-- change this to simulate noise -->
-        </noise>
+          <stddev>0.00</stddev>
+        </noise-->
         </plugin>
     </gazebo>

File: model/ft_sensor.urdf.xacro (robot description, xacro)
@@ -12,16 +12,16 @@
 		</joint>
 		<link name="${name}_${type}_base">
-			<insert_block name="nano17"/>
+			<insert_block name="ati_gamma"/>
 		</link>
-		<joint name="${parent}_${name}_measure_joint" type="revolute">
-			<insert_block name="nano17_measure_frame"/>
+	    <link name="${name}_${type}_measure">
+			<insert_block name="ati_gamma_platform"/>
+		</link>
+		<joint name="${parent}_${name}_measure_joint" type="fixed">
+		    <origin xyz="0 0 0.0165" rpy="0 0 0"/>
 			<parent link="${name}_${type}_base"/>
 			<child link="${name}_${type}_measure"/>
-			<limit lower="0" upper="0" effort="100" velocity="100"/>
-			<axis xyz="0 0 1" />
+			<!--limit lower="-0.00001" upper="0.00001" effort="100" velocity="100"/>
+			<axis xyz="0 0 1" /-->
 		</joint>
-		<link name="${name}_${type}_measure">
-			<insert_block name="nano17_platform"/>
-		</link>
         <xacro:ft_sensor_gazebo name="${name}" parent="${parent}" type="${type}"/>
 	</xacro:macro>

File: model/models.urdf.xacro (robot description, xacro)
@@ -63,3 +63,47 @@
 		<origin xyz="0 0 0.0145" rpy="0 0 0"/>
 	</xacro:property>
+	<xacro:property name="ati_gamma_platform">
+			<inertial>
+				<mass value="0.002"/>
+				<origin xyz="0 0 0.0025"  />
+				<xacro:cylinder_inertia_def radius="0.0377" length="0.005" mass="0.002"/>
+			</inertial>
+			<visual>
+				<!-- origin xyz="0 0 0.00725" rpy="0 0 0"/ -->
+				<origin xyz="0 0 0.0025" rpy="0 0 0"/>
+				<geometry>
+					<cylinder radius="0.0377" length="0.005"/>
+				</geometry>
+			</visual>
+			<collision>
+				<origin xyz="0 0 0.0025" rpy="0 0 0"/>
+				<geometry>
+					<cylinder radius="0.0377" length="0.005"/>
+				</geometry>
+			</collision>
+	</xacro:property>
+	<xacro:property name="ati_gamma_measure_frame">
+		<origin xyz="0 0 0.0165" rpy="0 0 0"/>
+	</xacro:property>
+	<xacro:property name="ati_gamma">
+			<inertial>
+				<mass value="0.255"/>
+				<origin xyz="0 0 0.0165"  />
+				<xacro:cylinder_inertia_def radius="0.0377" length="0.033" mass="0.255"/>
+			</inertial>
+			<visual>
+				<!-- origin xyz="0 0 0.00725" rpy="0 0 0"/ -->
+				<origin xyz="0 0 0" rpy="0 0 0"/>
+				<geometry>
+					<cylinder radius="0.0377" length="0.033"/>
+					<!--mesh filename="package://force_torque_sensor/model/meshes/ati_gamma.stl"/-->
+				</geometry>
+			</visual>
+			<collision>
+				<origin xyz="0 0 0.0165" rpy="0 0 0"/>
+				<geometry>
+					<cylinder radius="0.0377" length="0.033"/>
+				</geometry>
+			</collision>
+	</xacro:property>
 </robot>

File: robot/nano17.urdf.xacro (robot description, xacro)
@@ -4,5 +4,5 @@
 	<xacro:include filename="$(find force_torque_sensor)/model/ft_sensor.urdf.xacro"/>
 	<link name="world"/>
-	<xacro:ft_sensor parent="world" name="my_sensor" type="nano17">
+	<xacro:ft_sensor parent="world" name="my_sensor" type="ati_gamma">
 		<origin xyz="0 0 0" rpy="0 0 0"/>
 	</xacro:ft_sensor>
